Commit message: update

File: hurricane_description/urdf/gazebo.xacro (robot description, xacro)
@@ -8,9 +8,9 @@
             <odometryFrame>odom</odometryFrame>
             <odometryRate>20.0</odometryRate>
-            <robotBaseFrame>base</robotBaseFrame>
+            <robotBaseFrame>base_link</robotBaseFrame>
         </plugin>
     </gazebo>
     <!-- 仿真雷达 -->
-    <gazebo reference="base_link">
+    <gazebo reference="trunk">
         <sensor name="lidar_sensor" type="ray">
             <pose>0 0 0.2 0 0 0</pose>

File: hurricane_description/urdf/robot.xacro (robot description, xacro)
@@ -20,4 +20,12 @@
         </joint>
     </xacro:if>
+    <!-- base_footprint is the root link for navigation -->
+    <link name="base_footprint">
+    </link>
+    <joint name="base_footprint_to_base_link" type="fixed">
+        <origin rpy="0 0 0" xyz="0 0 0.213"/>
+        <parent link="base_footprint"/>
+        <child link="base_link"/>
+    </joint>
     <link name="base_link">
         <visual>
@@ -63,12 +71,5 @@
     <link name="utlidar_lidar">
     </link>
-    <!-- Todo: NEed to account for the calf joint angle and projected height of the calf.. -->
-    <joint name="base_footprint_joint" type="fixed">
-        <parent link="trunk"/>
-        <child link="base_footprint"/>
-        <origin rpy="0 0 0" xyz="0.0 0.0 -0.213"/>
-    </joint>
-    <link name="base_footprint">
-    </link>
+    <!-- base_footprint joint moved to top of file -->
     <joint name="imu_joint" type="fixed">
         <parent link="trunk"/>
